File: PCB/pump.sch (EAGLE design)
At the start: 16 parts, among them U1 ARDUINOR3-BPLACE, X1 HD44780LCD-1602

Commit message: Finished PCB
Parts:
- added JP14, JP15, JP16, JP17: (no value), adafruit:PINHD-1X1
Connections:
- new net N$1: JP15.1, JP6.2
- new net N$6: JP4.1, U1.D3
- net N$5: now also JP17.1
- net VSS: now also JP14.1, JP16.1; no longer JP6.2
